File: samples/m5/kicad/shapones_atoms3.kicad_sch (KiCad schematic)
At the start: 45 parts, among them J1 Micro_SD_Card, SW1 A, SW2 B, SW3 SELECT, SW4 START, SW5 UP, SW6 DOWN, SW7 LEFT, SW8 RIGHT, U1 AtomS3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

Commit message: wip: state saving
Parts:
- removed R10, R12, R16, R18, R6: 10k, symbol Device:R_Small
- R11, R17, R5: value 10k -> 22k
- R14, R15, R19, R8, R9: value 10k -> 4.7k
Connections:
- net GND: now also R11.2, R17.2, R5.2
Other:
- moved on the sheet: R13, R14, R20, R7, R8
